File: 01-kanto/01-MAIN/01-MAIN.kicad_pcb (KiCad board)
At the start: 2 copper layers, 80 x 100 mm, 114 parts, among them J1 LiDAR, J10 Loadcell_L, J11 Loadcell_R, J14 MG90S_L, J15 MG90_R, J4 CAM_LED_L, J5 CAM_LED_R, J6 USB_C_Receptacle_USB2.0_16P, J9 RPi, Q1 Q_PMOS_GDS, Q2 Q_PMOS_GDS, Q3 Q_PMOS_GDS, Q5 Q_PMOS_GDS, Q6 NPN, Q7 PNP, SW1 SW_SPST, SW2 SW_Push, SW3 SW_Push, SW4 SW_Push, SW6 SW_Push, SW7 SW_Push, U1 M51957B, U10 TPS5430DDA, U11 AMS1117-3.3, U12 TPS5430DDA, U2 MAX485E, U3 STM32F446RETx, U4 TPS5430DDA, U6 OKL-T/6-W12N-C, U7 BNO055, U8 CH340E, U9 LM358

Commit message: 配置した
Parts:
- removed D3, D4, D5, D6, D7, D8, D9: WS2812B, LED_SMD:LED_WS2812B_PLCC4_5.0x5.0mm_P3.2mm
- removed R41, R8, R9: 10k, Resistor_SMD:R_0402_1005Metric
- removed SW3, SW4: SW_Push, Button_Switch_THT:SW_PUSH_6mm
- added BT1: Battery, Connector_Wire:SolderWire-0.75sqmm_1x02_P7mm_D1.25mm_OD3.5mm, F.Cu at (214.4, 109.1)
- added J12: STS3032_F, Akizuki:Molex_SPOX_5268-03A_1x03_P2.50mm_Horizontal, F.Cu at (221.1, 67.7)
- added J13: STS3032_B, Akizuki:Molex_SPOX_5268-03A_1x03_P2.50mm_Horizontal, F.Cu at (222.4, 130.0)
- added J2: CAM_L, Akizuki:Grove_1x04, F.Cu at (155.8, 75.2)
- added J3: CAM_R, Akizuki:Grove_1x04, F.Cu at (224.8, 80.1)
- added J7: STS3032_F, Akizuki:Molex_SPOX_5268-03A_1x03_P2.50mm_Horizontal, F.Cu at (159.1, 63.8)
- added J8: STS3032_B, Akizuki:Molex_SPOX_5268-03A_1x03_P2.50mm_Horizontal, F.Cu at (157.6, 125.0)
- added MES1: Voltmeter_DC, Connector_JST:JST_XH_B2B-XH-A_1x02_P2.50mm_Vertical, F.Cu at (206.7, 115.4)
- added REF**: MountingHole_3.2mm_M3, MountingHole:MountingHole_3.2mm_M3, F.Cu at (223.0, 110.0)
- added REF**: MountingHole_3.2mm_M3, MountingHole:MountingHole_3.2mm_M3, F.Cu at (157.0, 55.0)
- added REF**: MountingHole_3.2mm_M3, MountingHole:MountingHole_3.2mm_M3, F.Cu at (157.0, 110.0)
- added REF**: MountingHole_3.2mm_M3, MountingHole:MountingHole_3.2mm_M3, F.Cu at (223.0, 55.0)
- added SW5: SW_SPDT, Akizuki:Akizuki_3PSW, F.Cu at (173.5, 130.8)
- added U5: SSD1306, Akizuki:SSD1306, F.Cu at (190.2, 121.8)
- BZ1, C1, C10, C11, C12, C13, C14, C15, C16, C17, C18, C19, C2, C20, C21, C22, C23, C24, C25, C3, C4, C5, C6, C7, C8, D10, D11, D13, D14, J6, L1, L2, L3, Q1, Q2, Q3, Q5, Q6, Q7, R1, R11, R13, R14, R15, R16, R17, R18, R19, R2, R20, R21, R22, R23, R24, R25, R26, R27, R3, R30, R31, R32, R33, R36, R37, R38, R39, R4, R40, R42, R43, R5, U1, U10, U11, U12, U2, U3, U4, U6, U8, U9: moved to B.Cu
- D12: footprint LED_SMD:LED_1206_3216Metric -> LED_SMD:LED_0805_2012Metric; moved to B.Cu
- J4, J5: footprint Connector_JST:JST_XH_S3B-XH-A_1x03_P2.50mm_Horizontal -> Connector_JST:JST_PH_S3B-PH-K_1x03_P2.00mm_Horizontal
- J9: footprint Connector_JST:JST_XH_S6B-XH-A_1x06_P2.50mm_Horizontal -> Connector_JST:JST_XH_B6B-XH-A_1x06_P2.50mm_Vertical; moved to B.Cu
- moved C17 191.9 mm to (211.9, 143.6), turned to 180 degrees
- moved C16 190.8 mm to (211.0, 146.7), turned to 90 degrees
- moved C22 180.8 mm to (215.2, 71.5)
- moved C21 180.5 mm to (215.1, 73.6)
- moved R27 179.3 mm to (208.1, 143.4), turned to 180 degrees
- moved L2 179.2 mm to (194.3, 119.5), turned to -90 degrees
- moved C1 176.8 mm to (193.3, 135.5), turned to -90 degrees
- moved SW2 174.5 mm to (163.9, 134.2), turned to 90 degrees
- moved R25 174.3 mm to (202.7, 141.1), turned to 180 degrees
- moved R3 171.9 mm to (201.0, 128.7), turned to 180 degrees
- moved D12 171.9 mm to (202.9, 143.6), turned to 180 degrees
- moved L3 171.2 mm to (194.1, 93.2), turned to 180 degrees
- moved C15 169.8 mm to (204.5, 86.3), turned to 90 degrees
- moved C14 169.7 mm to (204.5, 81.9), turned to -90 degrees
- moved L1 169.7 mm to (191.7, 77.5), turned to 180 degrees
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Connections:
- D2 pad 2: Net-(D2-DOUT) -> unconnected-(D2-DOUT-Pad2)
Routing:
- net VDD: track 0.00 -> 23.0 mm
- net Net-(Q1-S): track 0.00 -> 20.2 mm
- net +3V3: track 0.00 -> 19.4 mm
- net +5V: track 0.00 -> 15.8 mm
- net Net-(Q1-G): track 0.00 -> 15.6 mm
- net Net-(D13-K): track 0.00 -> 14.9 mm
- net GND: track 0.00 -> 14.8 mm
- net Net-(Q5-D): track 0.00 -> 13.6 mm
- net Net-(D10-K): track 0.00 -> 12.2 mm
- net Net-(BT1-+): track 0.00 -> 11.6 mm
- net Net-(D14-K): track 0.00 -> 11.6 mm
- net Net-(Q7-E): track 0.00 -> 7.34 mm
- net Net-(U1-IN): track 0.00 -> 6.73 mm
- net Net-(U10-BOOT): track 0.00 -> 5.78 mm
- net Net-(U12-BOOT): track 0.00 -> 5.62 mm
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- added copper zone on B.Cu, net GND
- added copper zone on F.Cu, net GND

Commit message: 01-MAIN, 02-BOTTOM, 04-RPi totally completed
Parts:
- added G***: LOGO, Logo:tuton_logo, F.Cu at (222.1, 142.9)
- added G***: LOGO, Logo:st_logo, F.Cu at (190.0, 144.1)
- added G***: LOGO, Logo:jlcpcb_logo, F.Cu at (189.4, 138.8)
- added J16: Victim_LED, Connector_JST:JST_XH_B3B-XH-A_1x03_P2.50mm_Vertical, F.Cu at (154.5, 118.9)
- added R28: 1M, Resistor_SMD:R_0402_1005Metric, B.Cu at (185.2, 56.4)
- added R29: 1M, Resistor_SMD:R_0402_1005Metric, B.Cu at (185.2, 54.1)
- added R34: 1M, Resistor_SMD:R_0402_1005Metric, B.Cu at (193.9, 53.8)
- added R35: 1M, Resistor_SMD:R_0402_1005Metric, B.Cu at (193.9, 55.8)
- C9, R10, R12, R7: moved to B.Cu
- moved J13 66.1 mm to (156.3, 127.0), turned to -90 degrees
- moved J7 64.5 mm to (223.5, 67.3), turned to 90 degrees
- moved J12 63.2 mm to (223.5, 130.8)
- moved J8 62.7 mm to (156.3, 62.3)
- moved U8 32.5 mm to (183.6, 136.4), turned to 90 degrees
- moved C16 31.9 mm to (182.4, 132.6), turned to 0 degrees
- moved C17 28.4 mm to (185.8, 132.3), turned to 90 degrees
- moved R27 24.8 mm to (183.4, 145.7), turned to 90 degrees
- moved D12 20.6 mm to (182.9, 148.6)
- moved R23 18.9 mm to (227.1, 84.6), turned to 0 degrees
- moved R22 15.8 mm to (225.0, 84.6), turned to 0 degrees
- moved R30 14.5 mm to (184.0, 54.1), turned to -90 degrees
- moved R31 14.5 mm to (184.0, 56.4), turned to 90 degrees
- moved R21 12.8 mm to (223.0, 84.6), turned to 0 degrees
- moved C9 11.1 mm to (170.8, 139.4), turned to 180 degrees
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Connections:
- R10 pad 2: SW4 -> SW2
- SW5 pad 2: SW4 -> SW2
- U3 pad 39: unconnected-(U3-PC8-Pad39) -> Victim_LED
- U3 pad 4: unconnected-(U3-PC15-Pad4) -> Loadcell_L
- U3 pad 40: unconnected-(U3-PC9-Pad40) -> MG90S_L
- U3 pad 41: unconnected-(U3-PA8-Pad41) -> CAM_LED_L
- U3 pad 45: unconnected-(U3-PA12-Pad45) -> SW2
- U3 pad 46: unconnected-(U3-PA13-Pad46) -> SW1
- U3 pad 49: unconnected-(U3-PA14-Pad49) -> LED
- U3 pad 50: unconnected-(U3-PA15-Pad50) -> Loadcell_R
- U3 pad 57: unconnected-(U3-PB5-Pad57) -> CAM_LED_R
- U3 pad 61: unconnected-(U3-PB8-Pad61) -> Buzzer
- U3 pad 62: unconnected-(U3-PB9-Pad62) -> MG90S_R
Routing:
- net +3V3: track 19.4 -> 309.0 mm, vias 0 -> 10
- net +5V: track 15.8 -> 291.7 mm, vias 0 -> 3
- net STS_SIG: track 0.00 -> 245.1 mm
- net NRST: track 0.00 -> 128.7 mm, vias 0 -> 2
- net MG90S_R: track 0.00 -> 127.6 mm, vias 0 -> 2
- net BOOT0: track 0.00 -> 124.5 mm, vias 0 -> 2
- net UART5_RX: track 0.00 -> 124.4 mm, vias 0 -> 2
- net UART5_TX: track 0.00 -> 121.1 mm, vias 0 -> 2
- net CAM_LED_R: track 0.00 -> 116.7 mm, vias 0 -> 4
- net UART1_RX: track 0.00 -> 115.3 mm, vias 0 -> 2
- net UART1_TX: track 0.00 -> 114.7 mm, vias 0 -> 2
- net Net-(J12-Pin_2): track 0.00 -> 109.0 mm
- net GND: track 14.8 -> 122.0 mm, vias 0 -> 459
- net Net-(J14-Pin_2): track 0.00 -> 94.2 mm, vias 0 -> 1
- net SW2: track 0.00 -> 88.6 mm, vias 0 -> 2
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- added copper zone on B.Cu, net VDD
- added copper zone on F.Cu, net VDD
Other:
- board text added: "+"
- board text added: "-"
- board text added: "1"
- board text added: "220uF"
- board text added: "3V3"
- board text added: "5V"
- board text added: "BNO055"
- board text added: "BOOT0"
- board text added: "CAM LED"
- board text added: "CH340E"
- board text added: "D"
- board text added: "FUSE"
- board text added: "G"
- board text added: "GND"
- board text added: "Kit Servo"
- board text added: "LIDAR"
- board text added: "LM358"
- board text added: "LiRX"
- board text added: "LiTX"
- board text added: "Loadcell"
- board text added: "M51957B"
- board text added: "NRST"
- board text added: "P Mosfet"
- board text added: "RX"
- board text added: "S"
- board text added: "SIG"
- board text added: "STS3032"
- board text added: "SW"
- board text added: "StRX"
- board text added: "StTX"
- board text added: "TX"
- board text added: "Trim"
- board text added: "Tuton 2026 Kanto 01-MAIN ver.1"
- board text added: "UnitV"
- board text added: "V"
- board text added: "VDD"
- board text added: "VictimLED"
- board text added: "|GND|"
- board text added: "←"
- board text added: "→"
