File: 01-kanto/01-MAIN/01-MAIN.kicad_sch (KiCad schematic)
At the start: 1 part, among them J1 Raspberry_Pi_4

Commit message: 基板は2枚だけさ
Parts:
- removed J1: Raspberry_Pi_4, symbol Connector:Raspberry_Pi_4
- added BT1: Battery, symbol Device:Battery
- added BZ1: Buzzer, symbol Device:Buzzer
- added C1: C, symbol Device:C
- added C2, C3, C4, C5, C6, C7, C9: 100n, symbol Device:C
- added C8: 4.7u, symbol Device:C
- added D1: LED, symbol Device:LED
- added D2, D3, D4, D5, D6, D7, D8, D9: WS2812B, LED_SMD:LED_WS2812B_PLCC4_5.0x5.0mm_P3.2mm, symbol LED:WS2812B
- added F1: 10A, symbol Device:Fuse
- added MES1: Voltmeter_DC, symbol Device:Voltmeter_DC
- added Q1, Q2, Q3, Q4: PMOS, symbol Simulation_SPICE:PMOS
- added R1, R2, R5: 100k, symbol Device:R
- added R10, R11, R12, R13, R14, R4, R7, R8, R9: 10k, symbol Device:R
- added R3: 78k, symbol Device:R
- added R6: R, symbol Device:R
- added SW1: SW_SPST, symbol Switch:SW_SPST
- added SW2, SW3, SW4, SW6, SW7: SW_Push, symbol Switch:SW_Push
- added SW5: SW_SPDT, symbol Switch:SW_SPDT
- added U1: ~, symbol akizuki:M51957BFP
- added U2: STM32F103C8Tx, Package_QFP:LQFP-48_7x7mm_P0.5mm, symbol MCU_ST_STM32F1:STM32F103C8Tx
- added U3: STM32F446RETx, Package_QFP:LQFP-64_10x10mm_P0.5mm, symbol MCU_ST_STM32F4:STM32F446RETx
Connections:
- new net: Q3.3 (S), Q4.3 (S), R3.1, R5.1, U1.7 (VIN)
- new net: R3.2, R4.1, U1.2 (IN)
- new net: D1.2 (A), R6.2
- new net: Q4.2 (G), R5.2, U1.6 (OUT)
- new net: D6.2 (DOUT), D7.4 (DIN)
- new net: D5.2 (DOUT), D6.4 (DIN)
- new net: D4.2 (DOUT), D5.4 (DIN)
- new net: D3.2 (DOUT), D4.4 (DIN)
- new net: D2.2 (DOUT), D3.4 (DIN)
- new net: R11.1, U2.20 (PB2)
- new net: Q2.2 (G), Q3.2 (G), R2.2, SW1.2 (B)
- new net: F1.2, Q1.1 (D), R1.1
- new net: C1.1, U1.5 (Cd)
- new net: Q2.1 (D), Q3.1 (D)
- new net: Q1.3 (S), Q2.3 (S), R2.1
- new net: U3.18 (VSS), U3.31 (VSS), U3.47 (VSS), U3.63 (VSS)
- new net: BT1.1 (+), F1.1
- new net: D8.2 (DOUT), D9.4 (DIN)
- new net: D7.2 (DOUT), D8.4 (DIN)
- new net +3V3: C2.1, C3.1, C4.1, C5.1, C6.1, C7.1, C8.1, R10.1, R13.2, R14.2, R7.1, R8.1, R9.1, SW7.1, U2.1 (VBAT), U2.24 (VDD), U2.36 (VDD), U2.48 (VDD), U2.9 (VDDA)
- new net +5V: D2.1 (VDD), D3.1 (VDD), D4.1 (VDD), D5.1 (VDD), D6.1 (VDD), D7.1 (VDD), D8.1 (VDD), D9.1 (VDD)
- new net BOOT0: R12.1, SW7.2, U2.44 (BOOT0)
- new net Buzzer: BZ1.1 (+)
- new net GND: BT1.2 (-), BZ1.2 (-), C1.2, C2.2, C3.2, C4.2, C5.2, C6.2, C7.2, C8.2, C9.2, D1.1 (K), D2.3 (VSS), D3.3 (VSS), D4.3 (VSS), D5.3 (VSS), D6.3 (VSS), D7.3 (VSS), D8.3 (VSS), D9.3 (VSS), MES1.1 (-), Q1.2 (G), R1.2, R11.2, R12.2, R4.2, SW1.1 (A), SW2.2, SW3.2, SW4.2, SW5.3 (C), SW6.1, U1.4 (GND), U2.23 (VSS), U2.35 (VSS), U2.47 (VSS), U2.8 (VSSA)
- new net LED: D2.4 (DIN)
- new net NRST: C9.1, SW6.2, U2.7 (NRST)
- new net SCL: R13.1, U2.42 (PB6)
- new net SDA: R14.1, U2.43 (PB7)
- new net SW1: R7.2, SW2.1
- new net SW2: R8.2, SW3.1
- new net SW3: R9.2, SW4.1
- new net SW4: R10.2, SW5.2 (B)
- new net UART1_RX: U2.31 (PA10)
- new net UART1_TX: U2.30 (PA9)
- new net VDD: MES1.2 (+), Q4.1 (D), R6.1
- no-connect marks 0 -> 7
Other:
- note added: "(R3+R4)/R4=88.8"
- note added: "LED"
- note added: "PWR"
- note added: "ハイサイドスイッチ＆逆流保護"
- note added: "低電圧防止 11.1V以下で強制遮断"
- note added: "逆接保護"
- note added: "電圧計"

Commit message: 02-BOTTOM PCBdesign completed
Parts:
- removed R11: 10k, symbol Device:R
- removed U2: STM32F103C8Tx, Package_QFP:LQFP-48_7x7mm_P0.5mm, symbol MCU_ST_STM32F1:STM32F103C8Tx
- added J1: LiDAR, symbol Connector_Generic:Conn_01x04
- added J2, J3: CAM_L, symbol Connector_Generic:Conn_01x04
Connections:
- net BOOT0: now also U3.60 (BOOT0)
- net NRST: now also U3.7 (NRST)
- net SCL: now also U3.37 (PC6)
- net SDA: now also U3.38 (PC7)
- net UART1_RX: now also U3.43 (PA10)
- net UART1_TX: now also U3.42 (PA9)
- no-connect marks 7 -> 2

Commit message: フットプリント途中
Parts:
- removed D1: LED, symbol Device:LED
- removed Q1, Q2, Q3, Q4: PMOS, symbol Simulation_SPICE:PMOS
- removed R6: R, symbol Device:R
- added C10, C16, C17: 100n, Capacitor_SMD:C_0402_1005Metric, symbol Device:C
- added C11, C15, C18, C23: 10u, Capacitor_SMD:C_0805_2012Metric, symbol Device:C
- added C12, C19, C24: 10n, Capacitor_SMD:C_0402_1005Metric, symbol Device:C
- added C13, C20, C25: 220u, Capacitor_THT:CP_Radial_D6.3mm_P2.50mm, symbol Device:C
- added C14, C21, C22: 22u, Capacitor_SMD:C_0805_2012Metric, symbol Device:C
- added D10, D13, D14: SS34, Diode_SMD:D_SMA, symbol Diode:SS34
- added D11: LED_GREEN, LED_SMD:LED_0805_2012Metric, symbol Device:LED
- added D12: LED_YELLOW, LED_SMD:LED_1206_3216Metric, symbol Device:LED
- added J10: Loadcell_L, Connector_JST:JST_PH_S4B-PH-K_1x04_P2.00mm_Horizontal, symbol Connector_Generic:Conn_01x04
- added J11: Loadcell_R, Connector_JST:JST_PH_S4B-PH-K_1x04_P2.00mm_Horizontal, symbol Connector_Generic:Conn_01x04
- added J12, J7: STS3032_F, symbol Connector_Generic:Conn_01x03
- added J13, J8: STS3032_B, symbol Connector_Generic:Conn_01x03
- added J14: MG90S_L, Connector_PinHeader_2.54mm:PinHeader_1x03_P2.54mm_Horizontal, symbol Connector_Generic:Conn_01x03
- added J15: MG90_R, Connector_PinHeader_2.54mm:PinHeader_1x03_P2.54mm_Horizontal, symbol Connector_Generic:Conn_01x03
- added J4: CAM_LED_L, Connector_JST:JST_XH_S3B-XH-A_1x03_P2.50mm_Horizontal, symbol Connector_Generic:Conn_01x03
- added J5: CAM_LED_R, Connector_JST:JST_XH_S3B-XH-A_1x03_P2.50mm_Horizontal, symbol Connector_Generic:Conn_01x03
- added J6: USB_C_Receptacle_USB2.0_16P, Connector_USB:USB_C_Receptacle_GCT_USB4105-xx-A_16P_TopMnt_Horizontal, symbol Connector:USB_C_Receptacle_USB2.0_16P
- added J9: RPi, Connector_JST:JST_XH_S6B-XH-A_1x06_P2.50mm_Horizontal, symbol Connector_Generic:Conn_01x06
- added L1, L2, L3: 22uH, LCSC:FXL1040-220-M, symbol Device:L
- added Q1, Q2, Q3, Q5: Q_PMOS_GDS, Package_TO_SOT_THT:TO-251-3_Vertical, symbol Transistor_FET:Q_PMOS_GDS
- added Q6: NPN, Package_TO_SOT_SMD:SOT-23, symbol Simulation_SPICE:NPN
- added Q7: PNP, Package_TO_SOT_SMD:SOT-23, symbol Simulation_SPICE:PNP
- added R11, R15, R19, R37, R42: 2k2, Resistor_SMD:R_0402_1005Metric, symbol Device:R
- added R16: 7k5, Resistor_SMD:R_0603_1608Metric, symbol Device:R
- added R17: 20k, Resistor_SMD:R_0402_1005Metric, symbol Device:R
- added R18, R36, R38, R39, R41, R43: 10k, Resistor_SMD:R_0402_1005Metric, symbol Device:R
- added R20: 1k2, Resistor_SMD:R_0603_1608Metric, symbol Device:R
- added R21: 1k, Resistor_SMD:R_0402_1005Metric, symbol Device:R
- added R22, R30, R31, R32, R33: 330, Resistor_SMD:R_0402_1005Metric, symbol Device:R
- added R23: 10, Resistor_SMD:R_0402_1005Metric, symbol Device:R
- added R24, R26: 5.1k, Resistor_SMD:R_0402_1005Metric, symbol Device:R
- added R25, R27: 470, Resistor_SMD:R_0603_1608Metric, symbol Device:R
- added R28, R29, R34, R35: 1M, symbol Device:R
- added R40: 2.7k, Resistor_SMD:R_0603_1608Metric, symbol Device:R
- added SW8: SW_SPDT, symbol Switch:SW_SPDT
- added U10, U12, U4: TPS5430DDA, Package_SO:TI_SO-PowerPAD-8_ThermalVias, symbol Regulator_Switching:TPS5430DDA
- added U11: AMS1117-3.3, Package_TO_SOT_SMD:SOT-223-3_TabPin2, symbol Regulator_Linear:AMS1117-3.3
- added U2: MAX485E, Package_SO:SOIC-8_3.9x4.9mm_P1.27mm, symbol Interface_UART:MAX485E
- added U5: SSD1306, symbol akizuki:SSD1306
- added U6: OKL-T/6-W12N-C, Akizuki:OKL-T6-W12N-C-SMD, symbol akizuki:OKL-T/6-W12N-C
- added U7: BNO055, Akizuki:BNO055, symbol akizuki:AE-BNO055-BO
- added U8: CH340E, Package_SO:MSOP-10_3x3mm_P0.5mm, symbol Interface_USB:CH340E
- added U9: LM358, Package_SO:SOIC-8-1EP_3.9x4.9mm_P1.27mm_EP2.29x3mm, symbol Amplifier_Operational:LM358
- BZ1: footprint (none) -> Buzzer_Beeper:Buzzer_TDK_PS1240P02BT_D12.2mm_H6.5mm
- C1: value C -> 4n7; footprint (none) -> Capacitor_SMD:C_0402_1005Metric; LCSC (none) -> C1538
- C2, C3, C4, C5, C6, C7, C9: footprint (none) -> Capacitor_SMD:C_0402_1005Metric; LCSC (none) -> C1525
- C8: footprint (none) -> Capacitor_SMD:C_0402_1005Metric; LCSC (none) -> C23733
- F1: footprint (none) -> Akizuki:FUSE_3557-15
- J1: footprint (none) -> Connector_JST:JST_PH_S4B-PH-K_1x04_P2.00mm_Horizontal
- J3: value CAM_L -> CAM_R
- R1, R2: footprint (none) -> Resistor_SMD:R_0402_1005Metric; LCSC (none) -> C25741
- R10, R12, R13, R14, R7, R8, R9: footprint (none) -> Resistor_SMD:R_0402_1005Metric; LCSC (none) -> C25744
- R3: value 78k -> 13k; footprint (none) -> Resistor_SMD:R_0603_1608Metric; LCSC (none) -> C22797
- R4: value 10k -> 1k8; footprint (none) -> Resistor_SMD:R_0603_1608Metric; LCSC (none) -> C4177
- R5: value 100k -> 10k; footprint (none) -> Resistor_SMD:R_0402_1005Metric; LCSC (none) -> C25744
- SW1: footprint (none) -> Akizuki:AkizukiSmallRockerSwitchHorizontal
- SW2, SW3, SW4, SW6, SW7: footprint (none) -> Button_Switch_THT:SW_PUSH_6mm
- U1: value ~ -> M51957B; footprint (none) -> Akizuki:M51957B
Connections:
- net +3V3: now also U3.1 (VBAT), U3.13 (VDDA), U3.19 (VDD), U3.32 (VDD), U3.48 (VDD), U3.64 (VDD), C22.1, J10.4 (Pin_4), J11.4 (Pin_4), R41.1, U11.2 (VO), U5.2 (VCC), U7.1 (VIN), U9.8 (V+)
- net +5V: now also J1.1 (Pin_1), J2.3 (Pin_3), J3.3 (Pin_3), C10.2, C15.1, C16.2, C21.1, J4.1 (Pin_1), J5.1 (Pin_1), J9.1 (Pin_1), Q7.1 (C), R15.1, R20.1, U11.3 (VI), U2.8 (VCC), U6.4 (Vout), U6.5 (Sense), U8.7 (VCC)
- net GND: now also J1.3 (Pin_3), J2.4 (Pin_4), J3.4 (Pin_4), U3.12 (VSSA), U3.18 (VSS), U3.31 (VSS), U3.47 (VSS), U3.63 (VSS), C10.1, C11.2, C13.2, C14.2, C15.2, C16.1, C17.2, C18.2, C20.2, C21.2, C22.2, C23.2, C25.2, D10.2 (A), D13.2 (A), D14.2 (A), J10.1 (Pin_1), J11.1 (Pin_1), J12.3 (Pin_3), J13.3 (Pin_3), J14.3 (Pin_3), J15.3 (Pin_3), J4.3 (Pin_3), J5.3 (Pin_3), J6.A1 (GND), J6.A12 (GND), J6.B1 (GND), J6.B12 (GND), J7.3 (Pin_3), J8.3 (Pin_3), J9.6 (Pin_6), Q5.1 (G), Q6.3 (E), R11.2, R17.2, R19.2, R20.2, R23.2, R24.1, R25.2, R26.1, R27.2, R29.2, R34.2, R37.2, R38.2, R40.2, SW8.3 (C), U10.6 (GND), U10.9 (GNDPAD), U11.1 (GND), U12.6 (GND), U12.9 (GNDPAD), U2.5 (GND), U4.6 (GND), U4.9 (GNDPAD), U5.1 (GND), U6.1 (ON/OFF), U6.3 (GND), U6.7 (GND), U7.2 (GND), U8.3 (GND), U9.4 (V-)
- net SCL: now also U3.58 (PB6), U5.3 (SCL), U7.4 (SCL); no longer U3.37 (PC6)
- net SDA: now also U3.59 (PB7), U5.4 (SDA), U7.3 (SDA); no longer U3.38 (PC7)
- net UART1_RX: now also U8.8 (TXD)
- net UART1_TX: now also U8.9 (RXD)
- net VDD: now also C11.1, C14.1, C18.1, C23.1, Q3.2 (D), U10.7 (VIN), U12.7 (VIN), U4.7 (VIN), U6.2 (Vin)
- net at R3.1, R5.1, U1.7 (VIN): now also Q1.3 (S), Q3.3 (S), R42.1
- net at R5.2, U1.6 (OUT): now also R43.1
- net at R2.2, SW1.2 (B): now also Q1.1 (G), Q2.1 (G)
- net LiDAR_TX: now reaches J1.2 (Pin_2)
- net LiDAR_TX: now also J9.4 (Pin_4)
- net LiDAR_RX: now reaches J1.4 (Pin_4)
- net LiDAR_RX: now also J9.5 (Pin_5)
- net UART4_RX: now reaches J2.1 (Pin_1)
- net UART4_RX: now also U3.15 (PA1)
- net UART4_TX: now reaches J2.2 (Pin_2)
- net UART4_TX: now also U3.14 (PA0)
- net at F1.2, R1.1: now also Q5.2 (D)
- net at R2.1: now also Q2.3 (S), Q5.3 (S)
- net UART2_TX: now reaches U3.16 (PA2)
- net UART2_TX: now also J9.3 (Pin_3)
- net UART2_RX: now reaches U3.17 (PA3)
- net UART2_RX: now also J9.2 (Pin_2)
- net BOOT1: now reaches U3.28 (PB2)
- net BOOT1: now also R38.1
- net UART3_TX: now reaches U3.51 (PC10)
- net UART3_TX: now also R16.2, U2.4 (DI)
- net UART3_RX: now reaches U3.52 (PC11)
- net UART3_RX: now also U2.1 (RO)
- net UART5_TX: now reaches U3.53 (PC12)
- net UART5_TX: now also J3.2 (Pin_2)
- net UART5_RX: now reaches U3.54 (PD2)
- net UART5_RX: now also J3.1 (Pin_1)
- new net: D11.1 (K), R25.1
- new net: D11.2 (A), J6.A4 (VBUS), J6.A9 (VBUS), J6.B4 (VBUS), J6.B9 (VBUS)
- new net: J6.A5 (CC1), R26.2
- new net: J6.B5 (CC2), R24.2
- new net: Q3.1 (G), Q6.1 (C), R42.2
- new net: C13.1, J7.2 (Pin_2), J8.2 (Pin_2), L1.2, R18.1
- new net: Q1.2 (D), Q2.2 (D)
- new net: C25.1, J14.2 (Pin_2), J15.2 (Pin_2), L3.2, R39.1
- new net: R21.2, R22.1
- new net: R22.2, R23.1
- new net: J11.2 (Pin_2), R32.1
- new net: R32.2, R34.1, U9.5 (+)
- new net: R21.1, U6.6 (Trim)
- new net: D12.1 (K), R27.1
- new net: R11.1, R15.2, U2.7 (B)
- new net: C24.1, U12.1 (BOOT)
- new net: R39.2, R40.1, U12.4 (VSENSE)
- new net: C24.2, D14.1 (K), L3.1, U12.8 (PH)
- new net: D12.2 (A), U8.6 (TNOW)
- new net: Q7.3 (E), R17.1, U2.2 (~{RE}), U2.3 (DE)
- new net: C12.1, U4.1 (BOOT)
- new net: R18.2, R19.1, U4.4 (VSENSE)
- new net: C12.2, D10.1 (K), L1.1, U4.8 (PH)
- new net: R36.2, R37.1, U10.4 (VSENSE)
- new net: C19.1, U10.1 (BOOT)
- new net: C19.2, D13.1 (K), L2.1, U10.8 (PH)
- new net: J11.3 (Pin_3), R33.1
- new net: R33.2, R35.1, U9.6 (-)
- new net: Q6.2 (B), R43.2
- new net: C20.1, J12.2 (Pin_2), J13.2 (Pin_2), L2.2, R36.1
- new net: R28.1, R31.2, U9.2 (-)
- new net: R29.1, R30.2, U9.3 (+)
- new net: Q7.2 (B), R16.1
- new net: C17.1, U8.10 (V3)
- new net: J10.3 (Pin_3), R31.1
- new net: J10.2 (Pin_2), R30.1
- new net CAM_LED_L: J4.2 (Pin_2)
- new net CAM_LED_R: J5.2 (Pin_2)
- new net D+: J6.A6 (D+), J6.B6 (D+), U8.1 (UD+)
- new net D-: J6.A7 (D-), J6.B7 (D-), U8.2 (UD-)
- new net Loadcell_L: R28.2, U9.1
- new net Loadcell_R: R35.2, U9.7
- new net MG90S_L: J14.1 (Pin_1)
- new net MG90S_R: J15.1 (Pin_1)
- new net STS_SIG: J12.1 (Pin_1), J13.1 (Pin_1), J7.1 (Pin_1), J8.1 (Pin_1), U2.6 (A)
- new net SW5: R41.2, SW8.2 (B)
- new net UART6_RX: U3.38 (PC7)
- new net UART6_TX: U3.37 (PC6)
- no-connect marks 2 -> 17
Other:
- note added: "(R3+R4)/R4=8.88"
- note added: "Bumper"
- note added: "POWER"
- note added: "STM32F446RE"
- note added: "STS3032"
- note added: "UI"
- note removed: "(R3+R4)/R4=88.8"
- note removed: "LED"
- note removed: "PWR"
- moved on the sheet: BZ1, C2, C3, C4, C5, C6, C7, C8, C9, D2, D3, D4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

Commit message: 配置した
Parts:
- removed D3, D4, D5, D6, D7, D8, D9: WS2812B, LED_SMD:LED_WS2812B_PLCC4_5.0x5.0mm_P3.2mm, symbol LED:WS2812B
- removed R41, R8, R9: 10k, Resistor_SMD:R_0402_1005Metric, symbol Device:R
- removed SW3, SW4: SW_Push, Button_Switch_THT:SW_PUSH_6mm, symbol Switch:SW_Push
- removed SW8: SW_SPDT, symbol Switch:SW_SPDT
- BT1: footprint (none) -> Connector_Wire:SolderWire-0.75sqmm_1x02_P7mm_D1.25mm_OD3.5mm
- D12: footprint LED_SMD:LED_1206_3216Metric -> LED_SMD:LED_0805_2012Metric
- J12, J13, J7, J8: footprint (none) -> Akizuki:Molex_SPOX_5268-03A_1x03_P2.50mm_Horizontal
- J2, J3: footprint (none) -> Akizuki:Grove_1x04
- J4, J5: footprint Connector_JST:JST_XH_S3B-XH-A_1x03_P2.50mm_Horizontal -> Connector_JST:JST_PH_S3B-PH-K_1x03_P2.00mm_Horizontal
- J9: footprint Connector_JST:JST_XH_S6B-XH-A_1x06_P2.50mm_Horizontal -> Connector_JST:JST_XH_B6B-XH-A_1x06_P2.50mm_Vertical
- MES1: footprint (none) -> Connector_JST:JST_XH_B2B-XH-A_1x02_P2.50mm_Vertical
- SW5: footprint (none) -> Akizuki:Akizuki_3PSW
- U5: footprint (none) -> Akizuki:SSD1306
Connections:
- no-connect marks 17 -> 16
Other:
- moved on the sheet: J11, R28, R29, R32, R33, R34, R35, U9B

Commit message: 01-MAIN, 02-BOTTOM, 04-RPi totally completed
Parts:
- added J16: Victim_LED, Connector_JST:JST_XH_B3B-XH-A_1x03_P2.50mm_Vertical, symbol Connector_Generic:Conn_01x03
- R28, R29, R34, R35: footprint (none) -> Resistor_SMD:R_0402_1005Metric; LCSC (none) -> C26083
Connections:
- net SW4 is gone; now on net SW2: R10.2, SW5.2 (B)
- net +5V: now also J16.1 (Pin_1)
- net Buzzer: now also U3.61 (PB8)
- net CAM_LED_L: now also U3.41 (PA8)
- net CAM_LED_R: now also U3.57 (PB5)
- net GND: now also J16.3 (Pin_3)
- net LED: now also U3.49 (PA14)
- net Loadcell_L: now also U3.4 (PC15)
- net Loadcell_R: now also U3.50 (PA15)
- net MG90S_L: now also U3.40 (PC9)
- net MG90S_R: now also U3.62 (PB9)
- net SW1: now also U3.46 (PA13)
- net Victim_LED: now reaches U3.39 (PC8)
- net Victim_LED: now also J16.2 (Pin_2)
- net SW2: now reaches U3.45 (PA12)
